File: schematic2/schematic2.sch (KiCad schematic (older format))
At the start: 37 parts, among them J1 Barrel_Jack, K1 TIANBO_HJR_1-2C, P1 Conn_02x20_Odd_Even, Q1 BC547, Q2 BC557, Q3 BC547, Q4 BC547, U1 buck

Commit message: modified:   schematic2/schematic2.kicad_pcb new file:   schematic2/schematic2.pro modified:   schematic2/schematic2.sch
Parts:
- BT1: value 6x AA NiMh -> 6x AAA NiMh
- J2: renamed from J?; value Conn_01x05 -> I2C BUS; footprint (none) -> Connector_Molex:Molex_KK-254_AE-6410-05A_1x05_P2.54mm_Vertical
- R3: value 82R -> 120R
Other:
- note added: "CAN USE PWM HERE TO LOWER THE\nRELAY HOLD CURRENT SINCE RELAY\nIS HELD ON ALL THE TIME PI IS ON"
- note added: "JUMPER FOR NO AUTO\nPOWER OFF. STAY ON\nUNTIL BATTERY FLAT"
- note added: "R3 SHOULD BE ADJUSTED TO GIVE\nAPPROPRIATE CHARGING CURRENT\nFOR THE BATTERIES USED"
Changed lines of the file:
@@
 P 5250 3500
 F 0 "BT1" H 5350 3600 50  0000 L CNN
-F 1 "6x AA NiMh" H 5350 3500 50  0000 L CNN
+F 1 "6x AAA NiMh" H 5350 3500 50  0000 L CNN
 F 2 "Connector_Molex:Molex_KK-254_AE-6410-02A_1x02_P2.54mm_Vertical" V 5250 3560 50  0001 C CNN
 F 3 "" V 5250 3560 50  0001 C CNN
@@
 P 3100 1150
 F 0 "R3" V 3180 1150 50  0000 C CNN
-F 1 "82R" V 3100 1150 50  0000 C CNN
+F 1 "120R" V 3100 1150 50  0000 C CNN
 F 2 "Resistor_THT:R_Axial_DIN0204_L3.6mm_D1.6mm_P5.08mm_Horizontal" V 3030 1150 50  0001 C CNN
 F 3 "" H 3100 1150 50  0001 C CNN
@@
 	8200 4900 8200 6050
 Wire Wire Line
-	8200 6050 7500 6050
-Wire Wire Line
 	7500 6050 7500 6250
 Wire Wire Line
@@
 	10350 1650 10350 1350
 Wire Wire Line
-	7500 6050 6800 6050
-Wire Wire Line
 	6800 6050 6800 5650
 Connection ~ 7500 6050
 Wire Wire Line
 	6500 5450 6250 5450
-Wire Wire Line
-	7500 4450 7500 6050
 Wire Wire Line
 	5500 4800 5150 4800
@@
 Wire Wire Line
 	9150 4250 9500 4250
-$Comp
-L power:+3.3V #PWR?
-U 1 1 5B401F11
-P 10300 4050
-F 0 "#PWR?" H 10300 3900 50  0001 C CNN
-F 1 "+3.3V" H 10300 4190 50  0000 C CNN
-F 2 "" H 10300 4050 50  0000 C CNN
-F 3 "" H 10300 4050 50  0000 C CNN
-	1    10300 4050
-	1    0    0    -1
-$EndComp
 Text GLabel 10550 4250 2    45   Input ~ 0
 PI_P_SIG
@@
 PI_P_SIG
 $Comp
-L Connector_Generic:Conn_01x05 J?
+L Connector_Generic:Conn_01x05 J2
 U 1 1 5B40371B
 P -5100 3000
-F 0 "J?" H -5100 3300 50  0000 C CNN
-F 1 "Conn_01x05" H -5100 2700 50  0000 C CNN
-F 2 "" H -5100 3000 50  0001 C CNN
+F 0 "J2" H -5100 3300 50  0000 C CNN
+F 1 "I2C BUS" H -5100 2700 50  0000 C CNN
+F 2 "Connector_Molex:Molex_KK-254_AE-6410-05A_1x05_P2.54mm_Vertical" H -5100 3000 50  0001 C CNN
 F 3 "~" H -5100 3000 50  0001 C CNN
 	1    -5100 3000
@@
 	-3250 3200 -4900 3200
 Connection ~ -3250 3200
+Wire Wire Line
+	7500 6050 8200 6050
+Wire Wire Line
+	6800 6050 7500 6050
+Wire Wire Line
+	7500 4450 7500 6050
+Text Notes 9700 4650 0    50   ~ 0
+CAN USE PWM HERE TO LOWER THE\nRELAY HOLD CURRENT SINCE RELAY\nIS HELD ON ALL THE TIME PI IS ON
+Text Notes 2300 1550 0    50   ~ 0
+R3 SHOULD BE ADJUSTED TO GIVE\nAPPROPRIATE CHARGING CURRENT\nFOR THE BATTERIES USED
+Text Notes 9300 3250 0    50   ~ 0
+JUMPER FOR NO AUTO\nPOWER OFF.  STAY ON\nUNTIL BATTERY FLAT
 $EndSCHEMATC

Commit message: add fuse and logo.
Parts:
- added F1: Polyfuse, Fuse:Fuse_2816_7142Metric_Pad3.20x4.45mm_HandSolder, symbol Device:Polyfuse
Connections:
- wire segments 148 -> 149
Changed lines of the file:
@@
 L Connector:Barrel_Jack J1
 U 1 1 5B44C5FE
-P 1350 1750
-F 0 "J1" H 1350 1960 50  0000 C CNN
-F 1 "Barrel_Jack" H 1350 1550 50  0000 C CNN
-F 2 "Connector_BarrelJack:BarrelJack_Horizontal" H 1400 1710 50  0001 C CNN
-F 3 "~" H 1400 1710 50  0001 C CNN
-	1    1350 1750
+P 800 1750
+F 0 "J1" H 800 1960 50  0000 C CNN
+F 1 "Barrel_Jack" H 800 1550 50  0000 C CNN
+F 2 "Connector_BarrelJack:BarrelJack_Horizontal" H 850 1710 50  0001 C CNN
+F 3 "~" H 850 1710 50  0001 C CNN
+	1    800  1750
 	1    0    0    -1
 $EndComp
@@
 Wire Wire Line
 	1800 1650 1800 1350
-Wire Wire Line
-	1650 1850 1700 1850
 Wire Wire Line
 	1700 1850 1700 2050
@@
 Text Notes 9300 3250 0    50   ~ 0
 JUMPER FOR NO AUTO\nPOWER OFF.  STAY ON\nUNTIL BATTERY FLAT
+$Comp
+L Device:Polyfuse F1
+U 1 1 5B476954
+P 1500 1650
+F 0 "F1" V 1400 1650 50  0000 C CNN
+F 1 "Polyfuse" V 1600 1650 50  0000 C CNN
+F 2 "Fuse:Fuse_2816_7142Metric_Pad3.20x4.45mm_HandSolder" H 1550 1450 50  0001 L CNN
+F 3 "~" H 1500 1650 50  0001 C CNN
+	1    1500 1650
+	0    1    1    0
+$EndComp
+Wire Wire Line
+	1100 1650 1350 1650
+Wire Wire Line
+	1100 1850 1700 1850
 $EndSCHEMATC

Commit message: Change clock for discreets.
Parts:
- removed J2: I2C BUS, Connector_Molex:Molex_KK-254_AE-6410-05A_1x05_P2.54mm_Vertical, symbol Connector_Generic:Conn_01x05
- added BT2: 3x AAA NiMh, Battery:BatteryHolder_Keystone_2479_3xAAA, symbol Device:Battery
- added C1: C_Small, Capacitor_THT:C_Disc_D4.7mm_W2.5mm_P5.00mm, symbol Device:C_Small
- added R12, R13, R14, R15, R16: 4K7, Resistor_THT:R_Axial_DIN0204_L3.6mm_D1.6mm_P5.08mm_Horizontal, symbol Device:R
- added U2: DS3231M, Package_SO:SOIC-16W_7.5x10.3mm_P1.27mm, symbol Timer_RTC:DS3231M
- added U3: MCP1700-1202E_SOT89, Package_TO_SOT_SMD:SOT-89-3, symbol Regulator_Linear:MCP1700-1202E_SOT89
- BT1: value 6x AAA NiMh -> 3x AAA NiMh; footprint Connector_Molex:Molex_KK-254_AE-6410-02A_1x02_P2.54mm_Vertical -> Battery:BatteryHolder_Keystone_2479_3xAAA
Connections:
- net labels added: SCL1, SDA1
- wire segments 149 -> 184

Commit message: Convert blocks to sheets.
At this point only the schematic is changed.
Parts:
- removed C1: C_Small, Capacitor_THT:C_Disc_D4.7mm_W2.5mm_P5.00mm, symbol Device:C_Small
- removed R12, R13, R14, R15, R16: 4K7, Resistor_THT:R_Axial_DIN0204_L3.6mm_D1.6mm_P5.08mm_Horizontal, symbol Device:R
- removed U1: buck, Mikee:BUCK_MODULE_5V, symbol Mikes:buck
- removed U2: DS3231M, Package_SO:SOIC-16W_7.5x10.3mm_P1.27mm, symbol Timer_RTC:DS3231M
- removed U3: MCP1700-1202E_SOT89, Package_TO_SOT_SMD:SOT-89-3, symbol Regulator_Linear:MCP1700-1202E_SOT89
Connections:
- wire segments 184 -> 148

Commit message: Layout done.
Changed lines of the file:
@@
 $EndComp
 $Sheet
-S 5200 6650 800  500
+S 1300 2700 800  500
 U 5B4BA298
 F0 "Sheet5B4BA297" 40
 F1 "clock.sch" 40
-F2 "V0" I R 6000 6800 40
-F3 "GND" I R 6000 7050 40
-F4 "V3v3" I L 5200 6800 40
-F5 "SCL1" I L 5200 6950 40
-F6 "SDA1" B L 5200 7050 40
+F2 "V0" I R 2100 2850 40
+F3 "GND" I R 2100 3100 40
+F4 "V3v3" I L 1300 2850 40
+F5 "SCL1" I L 1300 3000 40
+F6 "SDA1" B L 1300 3100 40
 $EndSheet
 Wire Wire Line

Commit message: Put the prebuilt buck converter back.
It's cheaper and easier.
Parts:
- added U1: buck, Mikee:BUCK_MODULE_5V, symbol Mikes:buck
- D11: value LED -> OR
- D2: value LED -> G
- D8: value LED -> R
Connections:
- wire segments 148 -> 149
Changed lines of the file:
@@
 $Descr A4 11693 8268
 encoding utf-8
-Sheet 1 3
+Sheet 1 2
 Title ""
 Date "15 nov 2012"
@@
 Wire Wire Line
 	6300 2450 6300 1650
-Connection ~ 6300 1650
 $Comp
 L power:GND #PWR09
@@
 Wire Wire Line
 	7700 1650 8900 1650
-Connection ~ 7700 1650
 Wire Wire Line
 	10350 1650 10350 1350
@@
 P 6800 4450
 F 0 "D8" H 6800 4550 50  0000 C CNN
-F 1 "LED" H 6800 4350 50  0000 C CNN
+F 1 "R" H 6800 4350 50  0000 C CNN
 F 2 "LED_THT:LED_D3.0mm" H 6800 4450 50  0001 C CNN
 F 3 "~" H 6800 4450 50  0001 C CNN
@@
 P 9900 3500
 F 0 "D11" H 9900 3600 50  0000 C CNN
-F 1 "LED" H 9900 3400 50  0000 C CNN
+F 1 "OR" H 9900 3400 50  0000 C CNN
 F 2 "LED_THT:LED_D3.0mm" H 9900 3500 50  0001 C CNN
 F 3 "~" H 9900 3500 50  0001 C CNN
@@
 P 3000 2550
 F 0 "D2" H 3000 2650 50  0000 C CNN
-F 1 "LED" H 3000 2450 50  0000 C CNN
+F 1 "G" H 3000 2450 50  0000 C CNN
 F 2 "LED_THT:LED_D3.0mm" H 3000 2550 50  0001 C CNN
 F 3 "~" H 3000 2550 50  0001 C CNN
@@
 	7100 3100 7100 3050
 Connection ~ 6700 3100
-$Sheet
-S 6850 1550 500  350
-U 5B480DB5
-F0 "Sheet5B480DB4" 50
-F1 "buck.sch" 50
-F2 "Vin" I L 6850 1650 40
-F3 "GND" I L 6850 1800 40
-F4 "Vout" I R 7350 1650 40
-$EndSheet
-Wire Wire Line
-	6850 1800 6700 1800
-Wire Wire Line
-	6700 1800 6700 2050
-Wire Wire Line
-	6300 1650 6850 1650
-Wire Wire Line
-	7350 1650 7700 1650
 Text GLabel -4300 2900 0    40   BiDi ~ 0
 SDA1
@@
 Wire Wire Line
 	5850 3100 6700 3100
+$Comp
+L Mikes:buck U1
+U 1 1 5B498832
+P 7150 1750
+F 0 "U1" H 7050 1750 50  0000 C CNN
+F 1 "buck" H 7100 1650 50  0000 C CNN
+F 2 "Mikee:BUCK_MODULE_5V" H 6950 1650 50  0001 C CNN
+F 3 "" H 7150 1750 50  0001 C CNN
+	1    7150 1750
+	1    0    0    -1
+$EndComp
+Wire Wire Line
+	6700 2050 7450 2050
+Wire Wire Line
+	7450 2050 7450 1950
+Connection ~ 6700 2050
+Wire Wire Line
+	6700 1650 6300 1650
+Connection ~ 6300 1650
+Wire Wire Line
+	7450 1650 7700 1650
+Wire Wire Line
+	6700 1950 6700 2050
+Connection ~ 7700 1650
 $EndSCHEMATC

Commit message: Added EEPROM
Parts:
- added C1: 0.1uF, Capacitor_THT:C_Disc_D3.0mm_W1.6mm_P2.50mm, symbol hat-design-rescue:C
- added IC1: CAT24C32WI-GT3, Package_SO:SOIJ-8_5.3x5.3mm_P1.27mm, symbol hat-design-rescue:AT24CS32-MAHM
- added JP2: Jumper_NO_Small, Connector_PinHeader_2.54mm:PinHeader_1x02_P2.54mm_Vertical, symbol Device:Jumper_NO_Small
- added R1: 1K, Resistor_THT:R_Axial_DIN0204_L3.6mm_D1.6mm_P5.08mm_Horizontal, symbol hat-design-rescue:R
- added R2, R3: 4K7, Resistor_THT:R_Axial_DIN0204_L3.6mm_D1.6mm_P5.08mm_Horizontal, symbol Device:R
- renumbered BT2 to BT1, BT1 to BT2, R7 to R10, R8 to R11, R9 to R12, R10 to R13, R11 to R14, R1 to R4, R2 to R5, R3 to R6, R4 to R7, R5 to R8, R6 to R9
Connections:
- wire segments 149 -> 171

Commit message: Fix wrongly connected clock battery reg
Connections:
- wire segments 171 -> 176
Changed lines of the file:
@@
 F0 "Sheet5B4BA297" 40
 F1 "clock.sch" 40
-F2 "V0" I R 2650 3050 40
-F3 "GND" I R 2650 3300 40
-F4 "V3v3" I L 1850 3050 40
-F5 "SCL1" I L 1850 3200 40
-F6 "SDA1" B L 1850 3300 40
+F2 "GND" I R 2650 3300 40
+F3 "V3v3" I L 1850 3050 40
+F4 "SCL1" I L 1850 3200 40
+F5 "SDA1" B L 1850 3300 40
+F6 "VI" I R 2650 3000 50
 $EndSheet
 Wire Wire Line
@@
 	1    0    0    -1
 $EndComp
+Wire Wire Line
+	2650 3000 3150 3000
+Wire Wire Line
+	3150 3000 3150 3300
+Wire Wire Line
+	3150 3300 5150 3300
+Wire Wire Line
+	5150 3300 5150 3750
+Wire Wire Line
+	5150 3750 5800 3750
+Connection ~ 5800 3750
 $EndSCHEMATC
