File: schematic2/schematic2.sch (KiCad schematic (older format))
At the start: 44 parts, among them IC1 CAT24C32WI-GT3, J1 Barrel_Jack, K1 TIANBO_HJR_1-2C, P1 Conn_02x20_Odd_Even, Q1 BC547, Q2 BC557, Q3 BC547, Q4 BC547, U1 buck

Commit message: Fix wron wiring to clock.
Connections:
- wire segments 176 -> 182
Other:
- moved on the sheet: D10
Changed lines of the file:
@@
 EESchema Schematic File Version 4
 LIBS:schematic2-cache
-LIBS:hat-design-cache
 EELAYER 26 0
 EELAYER END
@@
 	7250 3300 7250 3250
 Wire Wire Line
-	7150 2650 6850 2650
-Wire Wire Line
 	6850 2650 6850 1850
 $Comp
@@
 Connection ~ 8750 4450
 Wire Wire Line
-	10350 4450 11100 4450
+	10100 4450 10150 4450
 $Comp
 L Device:Jumper_NO_Small JP1
@@
 L Diode:1N4148 D10
 U 1 1 5B3B451F
-P 10200 4450
-F 0 "D10" H 10200 4550 50  0000 C CNN
-F 1 "1N4148" H 10200 4350 50  0000 C CNN
-F 2 "Diode_THT:D_DO-35_SOD27_P7.62mm_Horizontal" H 10200 4275 50  0001 C CNN
-F 3 "" H 10200 4450 50  0001 C CNN
-	1    10200 4450
+P 9950 4450
+F 0 "D10" H 9950 4550 50  0000 C CNN
+F 1 "1N4148" H 9950 4350 50  0000 C CNN
+F 2 "Diode_THT:D_DO-35_SOD27_P7.62mm_Horizontal" H 9950 4275 50  0001 C CNN
+F 3 "" H 9950 4450 50  0001 C CNN
+	1    9950 4450
 	1    0    0    -1
 $EndComp
@@
 Connection ~ 9700 4450
 Wire Wire Line
-	9700 4450 10050 4450
-Text GLabel 11100 4450 2    45   Input ~ 0
+	9700 4450 9800 4450
+Text GLabel 10150 4450 2    45   Input ~ 0
 PI_P_SIG
 Wire Wire Line
@@
 Wire Wire Line
 	8050 4650 8050 6250
-Text Notes 10250 4850 0    50   ~ 0
+Text Notes 9700 4850 0    50   ~ 0
 CAN USE PWM HERE TO LOWER THE\nRELAY HOLD CURRENT SINCE RELAY\nIS HELD ON ALL THE TIME PI IS ON
 Text Notes 2850 1750 0    50   ~ 0
 R3 SHOULD BE ADJUSTED TO GIVE\nAPPROPRIATE CHARGING CURRENT\nFOR THE BATTERIES USED
-Text Notes 9850 3450 0    50   ~ 0
+Text Notes 9500 3200 0    50   ~ 0
 JUMPER FOR NO AUTO\nPOWER OFF.  STAY ON\nUNTIL BATTERY FLAT
 $Comp
@@
 Wire Wire Line
 	2850 6550 3050 6550
-Connection ~ 1200 6700
 Text GLabel -4300 4100 0    60   Input ~ 0
 ID_SD
@@
 	5150 3750 5800 3750
 Connection ~ 5800 3750
+$Comp
+L power:GND #PWR0112
+U 1 1 5B5AD6CE
+P 2800 3400
+F 0 "#PWR0112" H 2800 3150 50  0001 C CNN
+F 1 "GND" H 2800 3250 50  0000 C CNN
+F 2 "" H 2800 3400 50  0001 C CNN
+F 3 "" H 2800 3400 50  0001 C CNN
+	1    2800 3400
+	1    0    0    -1
+$EndComp
+Wire Wire Line
+	2800 3400 2800 3300
+Wire Wire Line
+	2800 3300 2650 3300
+$Comp
+L power:+3.3V #PWR0113
+U 1 1 5B5B71E2
+P 1450 2900
+F 0 "#PWR0113" H 1450 2750 50  0001 C CNN
+F 1 "+3.3V" H 1450 3040 50  0000 C CNN
+F 2 "" H 1450 2900 50  0000 C CNN
+F 3 "" H 1450 2900 50  0000 C CNN
+	1    1450 2900
+	1    0    0    -1
+$EndComp
+Wire Wire Line
+	1450 2900 1450 3050
+Wire Wire Line
+	1450 3050 1850 3050
+Text GLabel 1750 3200 0    40   Input ~ 0
+SCL1
+Text GLabel 1750 3300 0    40   BiDi ~ 0
+SDA1
+Wire Wire Line
+	1750 3200 1850 3200
+Wire Wire Line
+	1850 3300 1750 3300
+Wire Wire Line
+	7150 2650 6850 2650
 $EndSCHEMATC

Commit message: Added sub sheet and some annotations. 	new file:   powermon.service
Parts:
- removed C1: 0.1uF, Capacitor_THT:C_Disc_D3.0mm_W1.6mm_P2.50mm, symbol hat-design-rescue:C
- removed IC1: CAT24C32WI-GT3, Package_SO:SOIJ-8_5.3x5.3mm_P1.27mm, symbol hat-design-rescue:AT24CS32-MAHM
- removed JP2: Jumper_NO_Small, Connector_PinHeader_2.54mm:PinHeader_1x02_P2.54mm_Vertical, symbol Device:Jumper_NO_Small
- removed R1: 1K, Resistor_THT:R_Axial_DIN0204_L3.6mm_D1.6mm_P5.08mm_Horizontal, symbol hat-design-rescue:R
- removed R2, R3: 4K7, Resistor_THT:R_Axial_DIN0204_L3.6mm_D1.6mm_P5.08mm_Horizontal, symbol Device:R
Connections:
- wire segments 182 -> 162
Other:
- note added: "Goes HIGH when Q1\nis OFF"
- note added: "Held ON by \ninput voltage."
- note added: "ON when Q1\nis OFF"
- moved on the sheet: P1

Commit message: Power the 3V line instead of the 5V.
Parts:
- removed BT1: 3x AAA NiMh, Battery:BatteryHolder_Keystone_2479_3xAAA, symbol Device:Battery
- removed F1: Polyfuse, Fuse:Fuse_2816_7142Metric_Pad3.20x4.45mm_HandSolder, symbol Device:Polyfuse
- removed J1: Barrel_Jack, Connector_BarrelJack:BarrelJack_Horizontal, symbol Connector:Barrel_Jack
- removed Q2: BC557, Package_TO_SOT_THT:TO-92_Inline, symbol Transistor_BJT:BC557
- removed U1: buck, Mikee:BUCK_MODULE_5V, symbol Mikes:buck
- added C3: 10uF, symbol Device:CP_Small
- added C4: 22uF, symbol Device:C_Small
- added Q2: 2N2907, Package_TO_SOT_THT:TO-92_Inline, symbol Transistor_BJT:2N3905
- added U1: AP1117-33, Package_TO_SOT_SMD:SOT-223-3_TabPin2, symbol Regulator_Linear:AP1117-33
- BT2: value 3x AAA NiMh -> 4x AAA NiMh
- R6: value 120R -> R
Connections:
- net labels removed: +9V
- wire segments 162 -> 169
Other:
- note added: "R6 SHOULD BE ADJUSTED TO GIVE\nAPPROPRIATE CHARGING CURRENT\nFOR THE BATTERIES USED AT\nAPPROX 0.05 CAPACITY"
- note added: "TO PI\nAPPROX 350mA"
- note removed: "R3 SHOULD BE ADJUSTED TO GIVE\nAPPROPRIATE CHARGING CURRENT\nFOR THE BATTERIES USED"
- moved on the sheet: BT2, D1, D10, D11, D2, D3, D4, D5, D6, D7, D8, D9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

Commit message: Re-layout.
Parts:
- removed MK1, MK2, MK3, MK4: M2.5, MountingHole:MountingHole_2.7mm_M2.5, symbol Mechanical:Mounting_Hole
- BT2: footprint Battery:BatteryHolder_Keystone_2479_3xAAA -> Connector_Molex:Molex_KK-254_AE-6410-02A_1x02_P2.54mm_Vertical
- C3, C4: footprint (none) -> Capacitor_THT:CP_Radial_D6.3mm_P2.50mm
Connections:
- wire segments 169 -> 170
Other:
- note added: "R6 SHOULD BE ADJUSTED TO GIVE\nAPPROPRIATE CHARGING CURRENT\nFOR THE BATTERIES USED, AT\nAPPROX 0.05 CAPACITY"
- note removed: "Mounting Holes"
- note removed: "R6 SHOULD BE ADJUSTED TO GIVE\nAPPROPRIATE CHARGING CURRENT\nFOR THE BATTERIES USED AT\nAPPROX 0.05 CAPACITY"
- moved on the sheet: BT2, D7
Changed lines of the file:
@@
 ID_SD and ID_SC PINS:\nThese pins are reserved for HAT ID EEPROM.\n\nAt boot time this I2C interface will be\ninterrogated to look for an EEPROM\nthat identifes the attached board and\nallows automagic setup of the GPIOs\n(and optionally, Linux drivers).\n\nDO NOT USE these pins for anything other\nthan attaching an I2C ID EEPROM. Leave\nunconnected if ID EEPROM not required.
-$Comp
-L Mechanical:Mounting_Hole MK1
-U 1 1 5834FB2E
-P 5450 6900
-F 0 "MK1" H 5550 6946 50  0000 L CNN
-F 1 "M2.5" H 5550 6855 50  0000 L CNN
-F 2 "MountingHole:MountingHole_2.7mm_M2.5" H 5450 6900 60  0001 C CNN
-F 3 "" H 5450 6900 60  0001 C CNN
-	1    5450 6900
-	1    0    0    -1
-$EndComp
-$Comp
-L Mechanical:Mounting_Hole MK3
-U 1 1 5834FBEF
-P 5900 6900
-F 0 "MK3" H 6000 6946 50  0000 L CNN
-F 1 "M2.5" H 6000 6855 50  0000 L CNN
-F 2 "MountingHole:MountingHole_2.7mm_M2.5" H 5900 6900 60  0001 C CNN
-F 3 "" H 5900 6900 60  0001 C CNN
-	1    5900 6900
-	1    0    0    -1
-$EndComp
-$Comp
-L Mechanical:Mounting_Hole MK2
-U 1 1 5834FC19
-P 5450 7100
-F 0 "MK2" H 5550 7146 50  0000 L CNN
-F 1 "M2.5" H 5550 7055 50  0000 L CNN
-F 2 "MountingHole:MountingHole_2.7mm_M2.5" H 5450 7100 60  0001 C CNN
-F 3 "" H 5450 7100 60  0001 C CNN
-	1    5450 7100
-	1    0    0    -1
-$EndComp
-$Comp
-L Mechanical:Mounting_Hole MK4
-U 1 1 5834FC4F
-P 5900 7100
-F 0 "MK4" H 6000 7146 50  0000 L CNN
-F 1 "M2.5" H 6000 7055 50  0000 L CNN
-F 2 "MountingHole:MountingHole_2.7mm_M2.5" H 5900 7100 60  0001 C CNN
-F 3 "" H 5900 7100 60  0001 C CNN
-	1    5900 7100
-	1    0    0    -1
-$EndComp
-Text Notes 5450 6750 0    50   ~ 0
-Mounting Holes
 $Comp
 L Device:Battery BT2
 U 1 1 5B3B41CD
-P 5600 3500
-F 0 "BT2" H 5700 3600 50  0000 L CNN
-F 1 "4x AAA NiMh" H 5700 3500 50  0000 L CNN
-F 2 "Battery:BatteryHolder_Keystone_2479_3xAAA" V 5600 3560 50  0001 C CNN
-F 3 "" V 5600 3560 50  0001 C CNN
-	1    5600 3500
+P 5600 2500
+F 0 "BT2" H 5700 2600 50  0000 L CNN
+F 1 "4x AAA NiMh" H 5700 2500 50  0000 L CNN
+F 2 "Connector_Molex:Molex_KK-254_AE-6410-02A_1x02_P2.54mm_Vertical" V 5600 2560 50  0001 C CNN
+F 3 "" V 5600 2560 50  0001 C CNN
+	1    5600 2500
 	1    0    0    -1
 $EndComp
@@
 L Diode:1N4001 D7
 U 1 1 5B3B494C
-P 6050 3100
-F 0 "D7" H 6050 3200 50  0000 C CNN
-F 1 "1N4001" H 6050 3000 50  0000 C CNN
-F 2 "Diode_THT:D_DO-41_SOD81_P10.16mm_Horizontal" H 6050 2925 50  0001 C CNN
-F 3 "" H 6050 3100 50  0001 C CNN
-	1    6050 3100
+P 6000 2050
+F 0 "D7" H 6000 2150 50  0000 C CNN
+F 1 "1N4001" H 6000 1950 50  0000 C CNN
+F 2 "Diode_THT:D_DO-41_SOD81_P10.16mm_Horizontal" H 6000 1875 50  0001 C CNN
+F 3 "" H 6000 2050 50  0001 C CNN
+	1    6000 2050
 	-1   0    0    1
 $EndComp
@@
 L power:GND #PWR0103
 U 1 1 5B3B8E03
-P 5600 4000
-F 0 "#PWR0103" H 5600 3750 50  0001 C CNN
-F 1 "GND" H 5600 3850 50  0000 C CNN
-F 2 "" H 5600 4000 50  0001 C CNN
-F 3 "" H 5600 4000 50  0001 C CNN
-	1    5600 4000
+P 5600 2900
+F 0 "#PWR0103" H 5600 2650 50  0001 C CNN
+F 1 "GND" H 5600 2750 50  0000 C CNN
+F 2 "" H 5600 2900 50  0001 C CNN
+F 3 "" H 5600 2900 50  0001 C CNN
+	1    5600 2900
 	1    0    0    -1
 $EndComp
@@
 CAN USE PWM HERE TO LOWER THE\nRELAY HOLD CURRENT SINCE RELAY\nIS HELD ON ALL THE TIME PI IS ON
 Text Notes 2650 1550 0    50   ~ 0
-R6 SHOULD BE ADJUSTED TO GIVE\nAPPROPRIATE CHARGING CURRENT\nFOR THE BATTERIES USED AT\nAPPROX 0.05 CAPACITY
+R6 SHOULD BE ADJUSTED TO GIVE\nAPPROPRIATE CHARGING CURRENT\nFOR THE BATTERIES USED, AT\nAPPROX 0.05 CAPACITY
 Text Notes 9300 3000 0    50   ~ 0
 JUMPER FOR NO AUTO\nPOWER OFF.  STAY ON\nUNTIL BATTERY FLAT
 Wire Wire Line
-	5600 4000 5600 3700
+	5600 2900 5600 2700
 Text GLabel -3150 2950 0    40   BiDi ~ 0
 SDA1
@@
 $EndComp
 $Sheet
-S 1650 2700 800  500
+S 4000 2800 800  500
 U 5B4BA298
 F0 "Sheet5B4BA297" 40
 F1 "clock.sch" 40
-F2 "GND" I R 2450 3100 40
-F3 "V3v3" I L 1650 2850 40
-F4 "SCL1" I L 1650 3000 40
-F5 "SDA1" B L 1650 3100 40
-F6 "VI" I R 2450 2800 50
+F2 "GND" I R 4800 3200 40
+F3 "V3v3" I L 4000 2950 40
+F4 "SCL1" I L 4000 3100 40
+F5 "SDA1" B L 4000 3200 40
+F6 "VI" I R 4800 2900 50
 $EndSheet
 Text GLabel -3150 4150 0    60   BiDi ~ 0
@@
 ID_SC
 Wire Wire Line
-	2450 2800 2950 2800
-Wire Wire Line
-	2950 2800 2950 3100
-Connection ~ 5600 3100
+	4800 2900 5300 2900
+Wire Wire Line
+	5300 2900 5300 3200
+Connection ~ 5600 2050
 $Comp
 L power:GND #PWR0112
 U 1 1 5B5AD6CE
-P 2600 3200
-F 0 "#PWR0112" H 2600 2950 50  0001 C CNN
-F 1 "GND" H 2600 3050 50  0000 C CNN
-F 2 "" H 2600 3200 50  0001 C CNN
-F 3 "" H 2600 3200 50  0001 C CNN
-	1    2600 3200
-	1    0    0    -1
-$EndComp
-Wire Wire Line
-	2600 3200 2600 3100
-Wire Wire Line
-	2600 3100 2450 3100
+P 4950 3300
+F 0 "#PWR0112" H 4950 3050 50  0001 C CNN
+F 1 "GND" H 4950 3150 50  0000 C CNN
+F 2 "" H 4950 3300 50  0001 C CNN
+F 3 "" H 4950 3300 50  0001 C CNN
+	1    4950 3300
+	1    0    0    -1
+$EndComp
+Wire Wire Line
+	4950 3300 4950 3200
+Wire Wire Line
+	4950 3200 4800 3200
 $Comp
 L power:+3.3V #PWR0113
 U 1 1 5B5B71E2
-P 1250 2700
-F 0 "#PWR0113" H 1250 2550 50  0001 C CNN
-F 1 "+3.3V" H 1250 2840 50  0000 C CNN
-F 2 "" H 1250 2700 50  0000 C CNN
-F 3 "" H 1250 2700 50  0000 C CNN
-	1    1250 2700
-	1    0    0    -1
-$EndComp
-Wire Wire Line
-	1250 2700 1250 2850
-Wire Wire Line
-	1250 2850 1650 2850
-Text GLabel 1550 3000 0    40   Input ~ 0
+P 3600 2800
+F 0 "#PWR0113" H 3600 2650 50  0001 C CNN
+F 1 "+3.3V" H 3600 2940 50  0000 C CNN
+F 2 "" H 3600 2800 50  0000 C CNN
+F 3 "" H 3600 2800 50  0000 C CNN
+	1    3600 2800
+	1    0    0    -1
+$EndComp
+Wire Wire Line
+	3600 2800 3600 2950
+Wire Wire Line
+	3600 2950 4000 2950
+Text GLabel 3900 3100 0    40   Input ~ 0
 SCL1
-Text GLabel 1550 3100 0    40   BiDi ~ 0
+Text GLabel 3900 3200 0    40   BiDi ~ 0
 SDA1
 Wire Wire Line
-	1550 3000 1650 3000
-Wire Wire Line
-	1650 3100 1550 3100
+	3900 3100 4000 3100
+Wire Wire Line
+	4000 3200 3900 3200
 $Sheet
 S 1200 6650 950  500
@@
 $EndComp
 Wire Wire Line
-	5600 1150 5600 3100
-Wire Wire Line
-	5900 3100 5600 3100
+	5600 1150 5600 2050
+Wire Wire Line
+	5850 2050 5600 2050
 Wire Wire Line
 	7450 3100 7450 3050
-Wire Wire Line
-	6200 3100 7050 3100
 Wire Wire Line
 	7050 3100 7450 3100
@@
 	7850 3050 7850 3200
 Connection ~ 7850 3200
-Wire Wire Line
-	7850 3200 8250 3200
 Wire Wire Line
 	8250 3200 8250 2900
@@
 $EndComp
 Wire Wire Line
-	2950 3100 5600 3100
-Wire Wire Line
-	5600 3300 5600 3100
+	5300 3200 7850 3200
+Wire Wire Line
+	5600 2300 5600 2050
 Wire Wire Line
 	7850 2450 8250 2450
@@
 F 0 "C4" H 8010 1170 50  0000 L CNN
 F 1 "22uF" H 8010 1020 50  0000 L CNN
-F 2 "" H 8000 1100 50  0001 C CNN
+F 2 "Capacitor_THT:CP_Radial_D6.3mm_P2.50mm" H 8000 1100 50  0001 C CNN
 F 3 "~" H 8000 1100 50  0001 C CNN
 	1    8000 1100
@@
 F 0 "C3" H 6560 1220 50  0000 L CNN
 F 1 "10uF" H 6560 1070 50  0000 L CNN
-F 2 "" H 6550 1150 50  0001 C CNN
+F 2 "Capacitor_THT:CP_Radial_D6.3mm_P2.50mm" H 6550 1150 50  0001 C CNN
 F 3 "~" H 6550 1150 50  0001 C CNN
 	1    6550 1150
@@
 Wire Wire Line
 	5900 1650 6800 1650
+Wire Wire Line
+	7850 3200 8250 3200
+Wire Wire Line
+	7050 3100 6150 3100
+Wire Wire Line
+	6150 3100 6150 2050
 $EndSCHEMATC

Commit message: Stuff;
Parts:
- added U?: MCP73831-4-OT, Package_TO_SOT_SMD:SOT-23-5, symbol Battery_Management:MCP73831-4-OT
Changed lines of the file:
@@
 Wire Wire Line
 	6150 3100 6150 2050
+$Comp
+L Battery_Management:MCP73831-4-OT U?
+U 1 1 5C1EB8E9
+P 2400 2350
+F 0 "U?" H 2100 2600 50  0000 L CNN
+F 1 "MCP73831-4-OT" H 2450 2600 50  0000 L CNN
+F 2 "Package_TO_SOT_SMD:SOT-23-5" H 2450 2100 50  0001 L CIN
+F 3 "http://ww1.microchip.com/downloads/en/DeviceDoc/20001984g.pdf" H 2250 2300 50  0001 C CNN
+	1    2400 2350
+	1    0    0    -1
+$EndComp
 $EndSCHEMATC

Commit message: modified:   doc/UPS.adoc modified:   firmware/src/powermon.py modified:   schematic2/schematic2-cache.lib modified:   schematic2/schematic2.kicad_pcb modified:   schematic2/schematic2.sch
Parts:
- removed C3: 10uF, Capacitor_THT:CP_Radial_D6.3mm_P2.50mm, symbol Device:CP_Small
- removed C4: 22uF, Capacitor_THT:CP_Radial_D6.3mm_P2.50mm, symbol Device:C_Small
- removed D5: 1N5404, Diode_THT:D_DO-41_SOD81_P10.16mm_Horizontal, symbol Diode:1N4001
- removed D6: 1N4148, Diode_THT:D_DO-35_SOD27_P7.62mm_Horizontal, symbol Diode:1N4148
- removed D7: 1N4001, Diode_THT:D_DO-41_SOD81_P10.16mm_Horizontal, symbol Diode:1N4001
- removed JP1: UPS, Connector_PinHeader_2.54mm:PinHeader_1x02_P2.54mm_Vertical, symbol Device:Jumper_NO_Small
- removed U?: MCP73831-4-OT, Package_TO_SOT_SMD:SOT-23-5, symbol Battery_Management:MCP73831-4-OT
- added D5, D6: BAT86, Diode_THT:D_DO-35_SOD27_P7.62mm_Horizontal, symbol Diode:BAT86
- added H1, H2: MountingHole, MountingHole:MountingHole_2.7mm, symbol Mechanical:MountingHole
- added R3: 4K7, Resistor_THT:R_Axial_DIN0204_L3.6mm_D1.6mm_P5.08mm_Horizontal, symbol Device:R
- added RV1: R_POT_TRIM, Potentiometer_THT:Potentiometer_Runtron_RM-065_Vertical, symbol Device:R_POT_TRIM
- D3: value 5V6 -> 3V0
- R9: value 8K2 -> 4K7
Connections:
- net +3V3: no longer D8.2 (A), R14.2, R7.2, U1.2 (VO)
- net +5V: now also D10.1 (K), D8.2 (A), D9.1 (K), K1.16, K1.8, K1.9, R13.1, R14.2, R7.2, U1.3 (VI)
- net POWER_FAIL: now also R3.2; no longer R9.2
- net at K1.13, K1.4: now also D6.1 (K)
- net at BT2.1 (+): now also D5.1 (K), D6.2 (A)
- net at Q2.3 (C): now also D5.2 (A)
- net Sheet5B4BA297/VI: no longer names the net of D9.2 (A), K1.1, Q4.1 (C)
- new net: R4.2, RV1.1
- new net: R5.1, RV1.3
- new net: Q1.2 (B), RV1.2
- new net: R3.1, R9.2
- new net V_BAT: U1.2 (VO)
Other:
- note added: "THE Vf OF THIS LED WILL AFFECT\nTHE BASE VOLTAGE OF Q1"
- note removed: "JUMPER FOR NO AUTO\nPOWER OFF. STAY ON\nUNTIL BATTERY FLAT"

Commit message: Mostly layout changes.
Parts:
- removed BT2: 4x AAA NiMh, Connector_Molex:Molex_KK-254_AE-6410-02A_1x02_P2.54mm_Vertical, symbol Device:Battery
- removed D1, D4: 1N4148, Diode_THT:D_DO-35_SOD27_P7.62mm_Horizontal, symbol Diode:1N4148
- removed D5, D6: BAT86, Diode_THT:D_DO-35_SOD27_P7.62mm_Horizontal, symbol Diode:BAT86
- removed Q2: 2N2907, Package_TO_SOT_THT:TO-92_Inline, symbol Transistor_BJT:2N3905
- removed R8, R9: 4K7, Resistor_THT:R_Axial_DIN0204_L3.6mm_D1.6mm_P5.08mm_Horizontal, symbol Device:R
- removed RV1: R_POT_TRIM, Potentiometer_THT:Potentiometer_Runtron_RM-065_Vertical, symbol Device:R_POT_TRIM
- removed U1: AP1117-33, Package_TO_SOT_SMD:SOT-223-3_TabPin2, symbol Regulator_Linear:AP1117-33
- added BT1, BT2: Battery_Cell, Connector_Molex:Molex_KK-254_AE-6410-02A_1x02_P2.54mm_Vertical, symbol Device:Battery_Cell
- added C1: 100n, Capacitor_THT:C_Disc_D4.3mm_W1.9mm_P5.00mm, symbol Device:C
- added C3: 100n, Capacitor_SMD:C_0805_2012Metric, symbol Device:C
- added D1: LED, LED_THT:LED_D3.0mm, symbol Device:LED
- added D12, D4: 3V6, Resistor_THT:R_Axial_DIN0207_L6.3mm_D2.5mm_P7.62mm_Horizontal, symbol Device:D_Zener
- added D13, D6: 1N4001, Diode_SMD:D_2010_5025Metric, symbol Device:D
- added D14, D15, D5, D7: 1N4001, Diode_SMD:D_2010_5025Metric, symbol Diode:1N4001
- added F1: Polyfuse, Fuse:Fuse_2816_7142Metric_Pad3.20x4.45mm_HandSolder, symbol Device:Polyfuse
- added H3, H5: MountingHole, MountingHole:MountingHole_3.2mm_M3, symbol Mechanical:MountingHole
- added J1: Barrel_Jack, Connector_BarrelJack:BarrelJack_Horizontal, symbol Connector:Barrel_Jack
- added Q2: DMP1045U, Package_TO_SOT_SMD:SOT-23, symbol Device:Q_PMOS_GDS
- added Q5: BC547, Package_TO_SOT_THT:TO-92L_Inline_Wide, symbol Transistor_BJT:BC547
- added R14: 2K2, Resistor_THT:R_Axial_DIN0204_L3.6mm_D1.6mm_P5.08mm_Horizontal, symbol Device:R
- added R15: 320R, Resistor_THT:R_Axial_DIN0204_L3.6mm_D1.6mm_P5.08mm_Horizontal, symbol Device:R
- added R5: 470R, Resistor_THT:R_Axial_DIN0204_L3.6mm_D1.6mm_P5.08mm_Horizontal, symbol Device:R
- added U1: buck, Mikee:BUCK_MODULE_5V, symbol Mikes:buck
- added U3: LM317_SOT-223, Package_TO_SOT_THT:TO-92L_Inline_Wide, symbol Regulator_Linear:LM317_SOT-223
- D10: footprint Diode_THT:D_DO-35_SOD27_P7.62mm_Horizontal -> Diode_SMD:D_2010_5025Metric
- D3: value 3V0 -> 5V6
- D9: footprint Diode_THT:D_DO-41_SOD81_P10.16mm_Horizontal -> Diode_SMD:D_2010_5025Metric
- H1, H2: footprint MountingHole:MountingHole_2.7mm -> MountingHole:MountingHole_3.2mm_M3
- R11: renamed from R14; value 4K7 -> 1K
- R3: value 4K7 -> 6R6; footprint Resistor_THT:R_Axial_DIN0204_L3.6mm_D1.6mm_P5.08mm_Horizontal -> Resistor_THT:R_Axial_DIN0207_L6.3mm_D2.5mm_P7.62mm_Horizontal
- R6: value R -> 8K2
- renumbered R4 to R1, R13 to R10, R5 to R2, R7 to R4, R10 to R7, R11 to R8, R12 to R9
Connections:
- net +5V: now also U1.4 (Vout+); no longer D10.1 (K), D2.2 (A), K1.8, K1.9, R10.1, R6.2
- net GND: now also R3.2, R6.1, C1.2, D15.2 (A), J1.2, Q5.3 (E), U1.2 (Vin-), U1.3 (Vout-); no longer D11.1 (K)
- net POWER_FAIL: now also R6.2; no longer R3.2
- net at D9.2 (A), K1.1, Q4.1 (C): now also D11.1 (K)
- net at K1.13: now also Q2.3 (S); no longer K1.4
- net at R1.2: now also Q1.2 (B), R2.1
- net at R3.1: now also BT2.2 (-), C3.2, D13.1 (K), D15.1 (K), Q5.2 (B), R15.2
- new net: D10.1 (K), R10.1
- new net: D7.1 (K), Q2.2 (D)
- new net: BT1.1 (+), C3.1, D4.1 (K), D7.2 (A), R5.1, U3.2 (VO)
- new net: F1.2, J1.1
- new net: D5.1 (K), K1.9, U1.1 (V+in)
- new net: D1.2 (A), R14.1, R5.2, U3.1 (ADJ)
- new net: C1.1, D14.1 (K), U3.3 (VI)
- new net: D1.1 (K), Q5.1 (C)
- new net: R14.2, R15.1
- new net: D4.2 (A), D6.2 (A)
- new net: D12.2 (A), D13.2 (A)
- new net +9V: D14.2 (A), D2.2 (A), D5.2 (A), F1.1, Q2.1 (G)
- new net CLK_BAT: BT1.2 (-), BT2.1 (+), D12.1 (K), D6.1 (K)
Other:
- note added: "0=OK, 1=POWER FAIL"
- note added: "LiPo Charging Section"
- note added: "POWER FAIL\nINDICATOR"
- note added: "POWER INDICATOR"
- note added: "Power Fail Detection"
- note added: "UPS ACTIVE\nINDICATOR"
- note removed: "CAN USE PWM HERE TO LOWER THE\nRELAY HOLD CURRENT SINCE RELAY\nIS HELD ON ALL THE TIME PI IS ON"
- note removed: "Goes HIGH when Q1\nis OFF"
- note removed: "Held ON by \ninput voltage."
- note removed: "ON when Q1\nis OFF"
- note removed: "R6 SHOULD BE ADJUSTED TO GIVE\nAPPROPRIATE CHARGING CURRENT\nFOR THE BATTERIES USED, AT\nAPPROX 0.05 CAPACITY"
- note removed: "THE Vf OF THIS LED WILL AFFECT\nTHE BASE VOLTAGE OF Q1"
- note removed: "TO PI\nAPPROX 350mA"
- moved on the sheet: D10, D11, D2, D3, D8, D9, P1, Q1, Q3, Q4, R1, R10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
