File: schematic2/schematic2.kicad_pcb (KiCad board)
At the start: 2 copper layers, 68.8 x 56 mm, 51 parts, among them J1 Barrel_Jack, K1 TIANBO_HJR_1-2C, P1 Conn_02x20_Odd_Even, Q1 BC547, Q2 DMP1045U, Q3 BC547, Q4 BC547, Q5 BC547, U1 buck, U2 DS3231M, U3 LM317_SOT-223

Commit message: modified:   schematic2.kicad_pcb
Other:
- board text added: "Pi UPS Rev 3"
- board text removed: "Pi UPS Rev 2"
Changed lines of the file:
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@@
     (mod_text_size 1 2)
     (mod_text_width 0.15)
-    (pad_size 1.7 2.5)
-    (pad_drill 0)
+    (pad_size 1.8 1.8)
+    (pad_drill 0.9)
     (pad_to_mask_clearance 0)
     (aux_axis_origin 200 150)
@@
     (descr "C, Disc series, Radial, pin pitch=5.00mm, , diameter*width=4.3*1.9mm^2, Capacitor, http://www.vishay.com/docs/45233/krseries.pdf")
     (tags "C Disc series Radial pin pitch 5.00mm  diameter 4.3mm width 1.9mm Capacitor")
-    (fp_text reference C1 (at 2.5 -2.2 90) (layer F.SilkS)
+    (fp_text reference C1 (at 4 -2 90) (layer F.SilkS)
       (effects (font (size 1 1) (thickness 0.15)))
     )
@@
     (tags capacitor)
     (attr smd)
-    (fp_text reference C3 (at 2.562499 0 90) (layer F.SilkS)
+    (fp_text reference C3 (at 0.062499 1.5 90) (layer F.SilkS)
       (effects (font (size 1 1) (thickness 0.15)))
     )
@@
     (tags capacitor)
     (attr smd)
-    (fp_text reference C2 (at 0 -1.65 90) (layer F.SilkS)
+    (fp_text reference C2 (at -0.0125 2 90) (layer F.SilkS)
       (effects (font (size 1 1) (thickness 0.15)))
     )
@@
     (tags diode)
     (attr smd)
-    (fp_text reference D14 (at 0 -2.28 90) (layer F.SilkS)
+    (fp_text reference D14 (at -4.25 0 180) (layer F.SilkS)
       (effects (font (size 1 1) (thickness 0.15)))
     )
@@
     (descr "Resistor, Axial_DIN0204 series, Axial, Horizontal, pin pitch=5.08mm, 0.167W, length*diameter=3.6*1.6mm^2, http://cdn-reichelt.de/documents/datenblatt/B400/1_4W%23YAG.pdf")
     (tags "Resistor Axial_DIN0204 series Axial Horizontal pin pitch 5.08mm 0.167W length 3.6mm diameter 1.6mm")
-    (fp_text reference R14 (at 2.54 -1.92) (layer F.SilkS)
+    (fp_text reference R14 (at -0.5 2) (layer F.SilkS)
       (effects (font (size 1 1) (thickness 0.15)))
     )
@@
     (descr "TO-92L leads in-line (large body variant of TO-92), also known as TO-226, wide, drill 0.75mm (see https://www.diodes.com/assets/Package-Files/TO92L.pdf and http://www.ti.com/lit/an/snoa059/snoa059.pdf)")
     (tags "TO-92L Inline Wide transistor")
-    (fp_text reference Q5 (at 2.54 -3.56 90) (layer F.SilkS)
+    (fp_text reference Q5 (at 4.04 2.5 90) (layer F.SilkS)
       (effects (font (size 1 1) (thickness 0.15)))
     )
@@
     (descr "LED, diameter 3.0mm, 2 pins")
     (tags "LED diameter 3.0mm 2 pins")
-    (fp_text reference D1 (at 1.27 -2.96) (layer F.SilkS)
+    (fp_text reference D1 (at 1.54 -3) (layer F.SilkS)
       (effects (font (size 1 1) (thickness 0.15)))
     )
@@
     (tags SOT-23)
     (attr smd)
-    (fp_text reference Q2 (at -2.5 0.95 180) (layer F.SilkS)
+    (fp_text reference Q2 (at -3 -0.05 180) (layer F.SilkS)
       (effects (font (size 1 1) (thickness 0.15)))
     )
@@
     (descr "Resistor, Axial_DIN0204 series, Axial, Horizontal, pin pitch=5.08mm, 0.167W, length*diameter=3.6*1.6mm^2, http://cdn-reichelt.de/documents/datenblatt/B400/1_4W%23YAG.pdf")
     (tags "Resistor Axial_DIN0204 series Axial Horizontal pin pitch 5.08mm 0.167W length 3.6mm diameter 1.6mm")
-    (fp_text reference R12 (at -2.3876 -0.1524 90) (layer F.SilkS)
+    (fp_text reference R12 (at 2.5 -2 90) (layer F.SilkS)
       (effects (font (size 1 1) (thickness 0.15)))
     )
@@
     (descr "Resistor, Axial_DIN0204 series, Axial, Horizontal, pin pitch=5.08mm, 0.167W, length*diameter=3.6*1.6mm^2, http://cdn-reichelt.de/documents/datenblatt/B400/1_4W%23YAG.pdf")
     (tags "Resistor Axial_DIN0204 series Axial Horizontal pin pitch 5.08mm 0.167W length 3.6mm diameter 1.6mm")
-    (fp_text reference R13 (at -2.3876 0.1016) (layer F.SilkS)
+    (fp_text reference R13 (at 4.5 -2) (layer F.SilkS)
       (effects (font (size 1 1) (thickness 0.15)))
     )
@@
     (tags "SOIC 1.27")
     (attr smd)
-    (fp_text reference U2 (at 2.286 -1.905) (layer F.SilkS)
+    (fp_text reference U2 (at 0.15 -6.135) (layer F.SilkS)
       (effects (font (size 1 1) (thickness 0.15)))
     )
@@
     (descr "TO-92 leads in-line, narrow, oval pads, drill 0.75mm (see NXP sot054_po.pdf)")
     (tags "to-92 sc-43 sc-43a sot54 PA33 transistor")
-    (fp_text reference Q3 (at 1.27 -3.56 180) (layer F.SilkS)
+    (fp_text reference Q3 (at -1.0296 -3.0848 180) (layer F.SilkS)
       (effects (font (size 1 1) (thickness 0.15)))
     )
@@
     (effects (font (size 2 1.5) (thickness 0.25)))
   )
-  (gr_text "Pi UPS Rev 2" (at 245.5 123 90) (layer F.SilkS)
+  (gr_text "Pi UPS Rev 3" (at 245.5 122.5 90) (layer F.SilkS)
     (effects (font (size 2 2) (thickness 0.22225)))
   )
