File: schematic2/clock.sch (KiCad schematic (older format))
At the start: 4 parts, among them U2 DS3231M

Commit message: Detail changes made from release note.
Parts:
- C2: footprint Capacitor_SMD:C_0805_2012Metric -> Capacitor_SMD:C_1206_3216Metric
Changed lines of the file:
@@
 Title "LiPo Pi UPS"
 Date "2021-08-11"
-Rev "3"
+Rev "4"
 Comp "MILLSTREAM COMPUTING"
 Comment1 ""
@@
 F 0 "C2" H 3650 4250 50  0000 L CNN
 F 1 "100nF" H 3600 4050 50  0000 L CNN
-F 2 "Capacitor_SMD:C_0805_2012Metric" H 3800 4150 50  0001 C CNN
+F 2 "Capacitor_SMD:C_1206_3216Metric" H 3800 4150 50  0001 C CNN
 F 3 "~" H 3800 4150 50  0001 C CNN
 	1    3800 4150
